File: usb-midi-shield.sch (EAGLE design)
At the start: 31 parts, among them IC1 ATMEGA32U2-TQFP, U1 ARDUINOR3NODIM

Commit message: changed to v1.1
Parts:
- removed MINI_USB: (no value), adafruit:USBMINIB
- added D6: GREEN, SparkFun-LED:LED-GREENLARGE
- added D7: RED, SparkFun-LED:LED-GREENLARGE
- added JP1: USB-MICROB, SparkFun-Connectors:USB-MICROB
- added PROG: AYZ0202AGRLC, SparkFun-Electromechanical:SWITCH-SPDTSMD
- added R7: 10k, microbuilder:RESISTOR0805
- added R8, R9: 1k, microbuilder:RESISTOR0805
- added SJ1, SJ2: SOLDERJUMPERTRACE, SparkFun-Passives:SOLDERJUMPERTRACE
- ICSP: value (none) -> AVR_SPI_PRG_6NS; device microbuilder:HEADER-2X3 -> SparkFun-Connectors:AVR_SPI_PRG_6NS
- LOGO1: value OSHW_LOGO_FILLX0200-NT -> OSHW_LOGO_FILLX0350-NT; device ohw-logo:OSHW_LOGO_FILLX0200-NT -> ohw-logo:OSHW_LOGO_FILLX0350-NT
Connections:
- net N$14 renamed MISO
- net N$17 renamed SCK
- net N$19 renamed MOSI
- net N$8 renamed ARDUINO_TX
- removed net N$24: HWB.2, IC1.PD7(INT7/HWB/AIN6/T0)
- removed net N$25: C1.P$2, IC1.XTAL1, R5.1, XTAL.2
- removed net N$6: IC1.D+, R1.2
- removed net N$7 (its old number): IC1.PD3(INT3/TXD1), U1.D0
- new net ARDUINO_RX: IC1.PD3(INT3/TXD1), PROG.O
- new net D-: IC1.D+, R2.2
- new net N$1: HWB.1, IC1.PD7(INT7/HWB/AIN6/T0), R7.1
- new net N$23: JP1.D-, R1.1, Z2.1
- new net N$29: R8.2, SJ1.2
- new net N$30: D7.A, R8.1
- new net N$32: R9.2, SJ2.2
- new net N$33: D6.A, R9.1
- new net N$34: SJ2.1, U1.D6
- new net N$36: SJ1.1, U1.D7
- new net N$37: PROG.P, U1.D0
- net GND: now also C4.P$2, D6.C, D7.C, HWB.2, JP1.GND; no longer C4.P$1, HWB.1, MINI_USB.GND
- net N$10: now also JP1.VBUS; no longer MINI_USB.VBUS
- net N$2: now also C1.P$2; no longer C2.P$2
- net N$3: now also JP1.D+; no longer MINI_USB.D-
- net N$4: now also C2.P$2, IC1.XTAL1, R5.1, XTAL.2; no longer IC1.D-, R2.2
- net N$5: now also IC1.D-, R1.2; no longer MINI_USB.D+, R1.1, Z2.1
- net N$9: now also C4.P$1; no longer C4.P$2
- net VCC: now also R7.2
Other:
- moved on the sheet: A0, A1, C1, C2, C3, C4, D1, D2, D3, D4, HWB, IC1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
